File: Schematics/LightController/LightingControl.sch (EAGLE design)
At the start: 18 parts, among them IC1 LM324N, X2 87758-0816

Commit message: updates to Light Schematics
Parts:
- removed X2: 87758-0816, con-molex:87758-0816
- added C5, C6, C7, C8: 3300uF, rcl:C-US025-024X044
- added IC2: LM324N, linear:LM324N
- added RF5, RF6, RF7, RF8: 2M, rcl:R-TRIMM3314G
- added RG5, RG6, RG7, RG8: 1M, rcl:R-US_0207/10
- added RIN4, RIN5, RIN6, RIN7: (no value), rcl:R-US_0207/10
- added VCC: 87758-0216, con-molex:87758-0216
- added VI, VO: 87758-1616, con-molex:87758-1616
Connections:
- removed net V03+: X2-5.S
- removed net V04+: X2-7.S
- removed net VI$1: C1.1, C2.1, C3.1, C4.1, RIN.1, RIN1.1, RIN2.1, RIN3.1
- new net N$10: IC2A.+IN, RIN4.2
- new net N$11: IC2B.-IN, RF6.S, RG6.2
- new net N$12: IC2B.+IN, RIN5.2
- new net N$13: IC2C.-IN, RF7.S, RG7.2
- new net N$14: IC2D.-IN, RF8.S, RG8.2
- new net N$15: IC2C.+IN, RIN6.2
- new net N$16: IC2D.+IN, RIN7.2
- new net N$9: IC2A.-IN, RF5.S, RG5.2
- new net V+: IC1P.V+, IC2P.V+
- new net VCC: VCC-1.S
- new net VI1: C1.1, RIN.1
- new net VI1+: VI-1.S
- new net VI2: C2.1, RIN1.1
- new net VI2+: VI-3.S
- new net VI3: C3.1, RIN2.1
- new net VI3+: VI-5.S
- new net VI4: C4.1, RIN3.1
- new net VI4+: VI-7.S
- new net VI5: C5.1, RIN4.1
- new net VI5+: VI-9.S
- new net VI6: C6.1, RIN5.1
- new net VI6+: VI-11.S
- new net VI7: C7.1, RIN6.1
- new net VI7+: VI-13.S
- new net VI8: C8.1, RIN7.1
- new net VI8+: VI-15.S
- new net VO5+: IC2A.OUT, RF5.E, VO-9.S
- new net VO6+: IC2B.OUT, RF6.E, VO-11.S
- new net VO7+: IC2C.OUT, RF7.E, VO-13.S
- new net VO8+: IC2D.OUT, RF8.E, VO-15.S
- net 0: now also C5.2, C6.2, C7.2, C8.2, RF5.A, RF6.A, RF7.A, RF8.A, RG5.1, RG6.1, RG7.1, RG8.1; no longer RG2.1
- net GND: now also IC1P.V-, IC2P.V-, RG2.1, VCC-2.S, VI-10.S, VI-12.S, VI-14.S, VI-16.S, VI-2.S, VI-4.S, VI-6.S, VI-8.S, VO-10.S, VO-12.S, VO-14.S, VO-16.S, VO-2.S, VO-4.S, VO-6.S, VO-8.S; no longer X2-2.S, X2-4.S, X2-6.S, X2-8.S
- net VO1+: now also VO-1.S; no longer X2-1.S
- net VO2+: now also VO-3.S; no longer X2-3.S
- net VO3+: now also VO-5.S
- net VO4+: now also VO-7.S
Other:
- moved on the sheet: IC1A
